Commit message: Add mapping.launch file. Add new RGBD camera.

File: catkin_ws/src/my_robot/urdf/my_robot.xacro (robot description, xacro)
@@ -183,3 +183,10 @@
     <topicName>/scan</topicName>
   </joint>
+  <joint name="camera_optical_joint" type="fixed">
+    <origin xyz="0 0 0" rpy="-1.5707 0 -1.5707"/>
+    <parent link="camera"/>
+    <child link="camera_link_optical"/>
+  </joint>
+  <link name="camera_link_optical">
+  </link>
 </robot>
